File: Controller/Controller Front/Controller Front/Controller Front.kicad_pcb (KiCad board)
At the start: 0 parts

Commit message: contoller and contoller front Rev 1
Other:
- board outline added: 217 x 128.5 mm
- copper layers 0 -> 2
Changed lines of the file:
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@@
 (kicad_pcb (version 20210228) (generator pcbnew)
+  (general
+    (thickness 1.6)
+  )
+  (paper "A4")
+  (layers
+    (0 "F.Cu" signal)
+    (31 "B.Cu" signal)
+    (32 "B.Adhes" user "B.Adhesive")
+    (33 "F.Adhes" user "F.Adhesive")
+    (34 "B.Paste" user)
+    (35 "F.Paste" user)
+    (36 "B.SilkS" user "B.Silkscreen")
+    (37 "F.SilkS" user "F.Silkscreen")
+    (38 "B.Mask" user)
+    (39 "F.Mask" user)
+    (40 "Dwgs.User" user "User.Drawings")
+    (41 "Cmts.User" user "User.Comments")
+    (42 "Eco1.User" user "User.Eco1")
+    (43 "Eco2.User" user "User.Eco2")
+    (44 "Edge.Cuts" user)
+    (45 "Margin" user)
+    (46 "B.CrtYd" user "B.Courtyard")
+    (47 "F.CrtYd" user "F.Courtyard")
+    (48 "B.Fab" user)
+    (49 "F.Fab" user)
+    (50 "User.1" user)
+    (51 "User.2" user)
+    (52 "User.3" user)
+    (53 "User.4" user)
+    (54 "User.5" user)
+    (55 "User.6" user)
+    (56 "User.7" user)
+    (57 "User.8" user)
+    (58 "User.9" user)
+  )
+  (setup
+    (pad_to_mask_clearance 0)
+    (pcbplotparams
+      (layerselection 0x00010fc_ffffffff)
+      (disableapertmacros false)
+      (usegerberextensions false)
+      (usegerberattributes true)
+      (usegerberadvancedattributes true)
+      (creategerberjobfile true)
+      (svguseinch false)
+      (svgprecision 6)
+      (excludeedgelayer true)
+      (plotframeref false)
+      (viasonmask false)
+      (mode 1)
+      (useauxorigin true)
+      (hpglpennumber 1)
+      (hpglpenspeed 20)
+      (hpglpendiameter 15.000000)
+      (dxfpolygonmode true)
+      (dxfimperialunits true)
+      (dxfusepcbnewfont true)
+      (psnegative false)
+      (psa4output false)
+      (plotreference true)
+      (plotvalue true)
+      (plotinvisibletext false)
+      (sketchpadsonfab false)
+      (subtractmaskfromsilk false)
+      (outputformat 1)
+      (mirror false)
+      (drillshape 0)
+      (scaleselection 1)
+      (outputdirectory "")
+    )
+  )
+  (net 0 "")
+  (gr_line (start 202.5 64) (end 249.5 64) (layer "Eco2.User") (width 0.15))
+  (gr_line (start 212.5 64) (end 212.5 69) (layer "Eco2.User") (width 0.15))
+  (gr_circle (center 240.5 83.5) (end 242.1 83.5) (layer "Eco2.User") (width 0.15) (fill none))
+  (gr_line (start 228.5 128.5) (end 228.5 83.5) (layer "Eco2.User") (width 0.15))
+  (gr_circle (center 244.5 69) (end 246.1 69) (layer "Eco2.User") (width 0.15) (fill none))
+  (gr_line (start 47.5 64) (end 32.5 64) (layer "Eco2.User") (width 0.15))
+  (gr_line (start 228.5 83.5) (end 240.5 83.5) (layer "Eco2.User") (width 0.15))
+  (gr_rect (start 220.5 79) (end 236.5 88) (layer "Eco2.User") (width 0.15) (fill none))
+  (gr_circle (center 244.5 145.5) (end 246.1 145.5) (layer "Eco2.User") (width 0.15) (fill none))
+  (gr_line (start 212.5 150.5) (end 212.5 145.5) (layer "Eco2.User") (width 0.15))
+  (gr_line (start 37.5 64) (end 37.5 69) (layer "Eco2.User") (width 0.15))
+  (gr_line (start 228.5 150.5) (end 228.5 128.5) (layer "Eco2.User") (width 0.15))
+  (gr_line (start 249.5 150.5) (end 237.5 150.5) (layer "Eco2.User") (width 0.15))
+  (gr_line (start 228.5 83.5) (end 216.5 83.5) (layer "Eco2.User") (width 0.15))
+  (gr_circle (center 212.5 145.5) (end 214.1 145.5) (layer "Eco2.User") (width 0.15) (fill none))
+  (gr_circle (center 228.5 128.5) (end 246 128.5) (layer "Eco2.User") (width 0.15) (fill none))
+  (gr_rect (start 32.5 43) (end 249.5 171.5) (layer "Eco2.User") (width 0.15) (fill none))
+  (gr_rect (start 47.5 64) (end 202.5 150.5) (layer "Eco2.User") (width 0.15) (fill none))
+  (gr_line (start 244.5 64) (end 244.5 69) (layer "Eco2.User") (width 0.15))
+  (gr_line (start 47.5 43) (end 47.5 64) (layer "Eco2.User") (width 0.15))
+  (gr_line (start 47.5 150.5) (end 32.5 150.5) (layer "Eco2.User") (width 0.15))
+  (gr_circle (center 212.5 69) (end 210.9 69) (layer "Eco2.User") (width 0.15) (fill none))
+  (gr_line (start 32.5 150.5) (end 36.5 150.5) (layer "Eco2.User") (width 0.15))
+  (gr_line (start 37.5 150.5) (end 37.5 145.5) (layer "Eco2.User") (width 0.15))
+  (gr_line (start 202.5 150.5) (end 249.5 150.5) (layer "Eco2.User") (width 0.15))
+  (gr_line (start 244.5 150.5) (end 244.5 145.5) (layer "Eco2.User") (width 0.15))
+  (gr_circle (center 37.5 69) (end 39.1 69) (layer "Eco2.User") (width 0.15) (fill none))
+  (gr_line (start 32.5 64) (end 35.5 64) (layer "Eco2.User") (width 0.15))
+  (gr_circle (center 216.5 83.5) (end 218.1 83.5) (layer "Eco2.User") (width 0.15) (fill none))
+  (gr_circle (center 228.5 128.5) (end 246 128.5) (layer "Edge.Cuts") (width 0.1) (fill none))
+  (gr_circle (center 141 46) (end 142.6 46) (layer "Edge.Cuts") (width 0.1) (fill none))
+  (gr_circle (center 141 168.5) (end 142.6 168.5) (layer "Edge.Cuts") (width 0.1) (fill none))
+  (gr_circle (center 37.5 69) (end 39.1 69) (layer "Edge.Cuts") (width 0.1) (fill none))
+  (gr_circle (center 244.5 168.5) (end 246.1 168.5) (layer "Edge.Cuts") (width 0.1) (fill none))
+  (gr_circle (center 37.5 46) (end 39.1 46) (layer "Edge.Cuts") (width 0.1) (fill none))
+  (gr_rect (start 249.5 171.5) (end 32.5 43) (layer "Edge.Cuts") (width 0.1) (fill none))
+  (gr_rect (start 47.5 64) (end 202.5 150.5) (layer "Edge.Cuts") (width 0.1) (fill none))
+  (gr_circle (center 244.5 145.5) (end 246.1 145.5) (layer "Edge.Cuts") (width 0.1) (fill none))
+  (gr_circle (center 37.5 168.5) (end 39.1 168.5) (layer "Edge.Cuts") (width 0.1) (fill none))
+  (gr_circle (center 37.5 145.5) (end 39.1 145.5) (layer "Edge.Cuts") (width 0.1) (fill none))
+  (gr_circle (center 244.5 46) (end 246.1 46) (layer "Edge.Cuts") (width 0.1) (fill none))
+  (gr_circle (center 212.5 145.5) (end 214.1 145.5) (layer "Edge.Cuts") (width 0.1) (fill none))
+  (gr_circle (center 240.5 83.5) (end 242.1 83.5) (layer "Edge.Cuts") (width 0.1) (fill none))
+  (gr_rect (start 220.5 79) (end 236.5 88) (layer "Edge.Cuts") (width 0.1) (fill none))
+  (gr_circle (center 212.5 69) (end 214.1 69) (layer "Edge.Cuts") (width 0.1) (fill none))
+  (gr_circle (center 216.5 83.5) (end 218.1 83.5) (layer "Edge.Cuts") (width 0.1) (fill none))
+  (gr_circle (center 244.5 69) (end 246.1 69) (layer "Edge.Cuts") (width 0.1) (fill none))
 )
