File: Controller/Controller Front/Controller Front/Controller Front.kicad_pcb (KiCad board)
At the start: 2 copper layers, 217 x 128.5 mm, 0 parts

Commit message: Rev 3 Pcb's
Routing:
- added copper zone on F.Cu, net (none)
Other:
- board text added: "Powersupply Controller Rev 2 By Arne Van den Broeck (Nortle)"
- board text added: "USB"
Changed lines of the file:
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@@
       (drillshape 0)
       (scaleselection 1)
-      (outputdirectory "")
+      (outputdirectory "Gerber/")
     )
   )
@@
   (gr_circle (center 216.5 83.5) (end 218.1 83.5) (layer "Edge.Cuts") (width 0.1) (fill none))
   (gr_circle (center 244.5 69) (end 246.1 69) (layer "Edge.Cuts") (width 0.1) (fill none))
+  (gr_text "USB" (at 228.6 77) (layer "F.SilkS")
+    (effects (font (size 2 2) (thickness 0.15)))
+  )
+  (gr_text "Powersupply Controller Rev 2\nBy Arne Van den Broeck (Nortle)" (at 192.8 47.8) (layer "F.SilkS")
+    (effects (font (size 2 2) (thickness 0.15)))
+  )
+  (zone (net 0) (net_name "") (layer "F.Cu") (hatch edge 0.508)
+    (connect_pads yes (clearance 0.508))
+    (min_thickness 0.254) (filled_areas_thickness no)
+    (fill yes (thermal_gap 0.508) (thermal_bridge_width 0.508) (smoothing fillet) (radius 1))
+    (polygon
+      (pts
+        (xy 249.6 171.6)
+        (xy 32.4 171.6)
+        (xy 32.4 42.8)
+        (xy 249.6 42.8)
+      )
+    )
+  )
 )
