File: Powerboard 1/PowerBoard 1/PowerBoard 1.kicad_pcb (KiCad board)
At the start: 2 copper layers, 118.7 x 100 mm, 155 parts, among them J1 Conn_01x03_Male, J2 Conn_01x03_Male, J3 Conn_01x03_Male, J4 Conn_01x03, J5 Conn_01x02_Male, J6 Conn_02x20_Counter_Clockwise, J7 Conn_01x01_Female, J8 Conn_01x01_Female, Q1 TP0610L, Q2 BC808, Q3 BC808, Q4 BC808, Q5 BC808, Q6 2N3904, Q7 2N3904, Q8 BC808, SW1 SW_Push, U1 ISO1540DR, U10 LM335Z, U11 TL062, U12 EL3H7-G, U13 EL3H7-G, U14 LT3083, U15 TL062, U16 LM334Z, U2 LT6657AHMS8-3, U3 LT8607, U4 STM32F303K8Tx, U5 LT3680, U6 M24C01-FDW, U7 LM334Z, U8 LM335Z, U9 LM334Z, Y1 8Mhz

Commit message: Rev 3 Pcb's
Parts:
- added D10: ss34, Diode_SMD:D_SMA_Handsoldering, F.Cu at (118.0, 85.0)
- added D11: ss34, Diode_SMD:D_SMA_Handsoldering, F.Cu at (99.0, 85.0)
- added D12: ss34, Diode_SMD:D_SMA_Handsoldering, F.Cu at (108.5, 85.0)
- added D9: ss34, Diode_SMD:D_SMA_Handsoldering, F.Cu at (89.5, 85.0)
- added J9: Conn_01x04, Connector_PinSocket_2.54mm:PinSocket_1x04_P2.54mm_Vertical, F.Cu at (153.0, 60.0)
- added R10: 10Kohm, Resistor_SMD:R_0805_2012Metric_Pad1.20x1.40mm_HandSolder, F.Cu at (152.5, 45.0)
- added R11: 20Kohm, Resistor_SMD:R_0805_2012Metric_Pad1.20x1.40mm_HandSolder, F.Cu at (108.5, 71.5)
- added R12: 20Kohm, Resistor_SMD:R_0805_2012Metric_Pad1.20x1.40mm_HandSolder, F.Cu at (119.5, 77.5)
- added R70: 20Kohm, Resistor_SMD:R_0805_2012Metric_Pad1.20x1.40mm_HandSolder, F.Cu at (119.5, 71.5)
- added R71: 8Kohm, Resistor_SMD:R_0805_2012Metric_Pad1.20x1.40mm_HandSolder, F.Cu at (117.5, 71.5)
- added R72: 2Kohm, Resistor_SMD:R_0805_2012Metric_Pad1.20x1.40mm_HandSolder, F.Cu at (120.2, 51.5)
- C11, C12: value 0.1µF -> 100nF
- C16: value 1uF Film -> 1uF
- C22: value 0.47µF -> 470nF
- C3: value 1pF -> 1uF
- C36: value 1µ -> 1uF
- Q1: footprint Package_TO_SOT_THT:TO-92L_Inline -> Package_TO_SOT_SMD:SOT-23
- Q2, Q3, Q4, Q5: value BC808 -> 2N3904
- Q6, Q7: footprint Package_TO_SOT_THT:TO-92_Inline -> Package_TO_SOT_SMD:SOT-23
- R31, R45, R60: value 20Kohm -> 8Kohm
- R32, R48, R55, R64: value 370ohm -> 800ohm
- R47: value 4Kohm -> 2Kohm
- moved R32 25.3 mm to (91.0, 82.0), turned to 180 degrees
- moved R48 18.0 mm to (119.5, 82.0), turned to 180 degrees
- moved R55 14.3 mm to (100.5, 82.0), turned to 180 degrees
- moved R64 13.7 mm to (110.0, 82.0), turned to 180 degrees
- moved Q4 13.1 mm to (103.5, 77.5)
- moved Q2 13.1 mm to (103.5, 71.5)
- moved R31 13.1 mm to (106.5, 71.5)
- moved R54 11.1 mm to (108.5, 77.5), turned to 90 degrees
- moved Q3 9.12 mm to (114.5, 77.5)
- moved R45 9.12 mm to (117.5, 77.5)
- moved Q5 9.03 mm to (114.5, 71.5)
- moved R60 7.24 mm to (106.5, 77.5)
- moved Q6 2.23 mm to (98.0, 43.5)
- moved U3 0.31 mm to (80.0, 54.5)
- moved C6 0.25 mm to (140.2, 32.5)
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Connections:
- Q2 pad 1: Net-(Q2-Pad1) -> GND
- Q2 pad 2: Vin -> Net-(Q2-Pad2)
- Q2 pad 3: Net-(Q2-Pad3) -> Net-(D9-Pad2)
- Q3 pad 1: Net-(Q3-Pad1) -> GND
- Q3 pad 2: Vin -> Net-(Q3-Pad2)
- Q3 pad 3: Net-(Q3-Pad3) -> Net-(D10-Pad2)
- Q4 pad 1: Net-(Q4-Pad1) -> GND
- Q4 pad 2: Vin -> Net-(Q4-Pad2)
- Q4 pad 3: Net-(Q4-Pad3) -> Net-(D11-Pad2)
- Q5 pad 1: Net-(Q5-Pad1) -> GND
- Q5 pad 2: Vin -> Net-(Q5-Pad2)
- Q5 pad 3: Net-(Q5-Pad3) -> Net-(D12-Pad2)
- R31 pad 2: Net-(Q2-Pad1) -> Net-(Q2-Pad2)
- R32 pad 2: Net-(Q2-Pad3) -> Vin
- R45 pad 2: Net-(Q3-Pad1) -> Net-(Q3-Pad2)
- R48 pad 2: Net-(Q3-Pad3) -> Vin
- R54 pad 1: Relay3 -> GND
- R54 pad 2: Net-(Q4-Pad1) -> Relay3
- R55 pad 2: Net-(Q4-Pad3) -> Vin
- R60 pad 1: Relay4 -> Relay3
- R60 pad 2: Net-(Q5-Pad1) -> Net-(Q4-Pad2)
- R64 pad 2: Net-(Q5-Pad3) -> Vin
- RL1 pad 2: GND -> Net-(D9-Pad2)
- RL2 pad 2: GND -> Net-(D10-Pad2)
- RL3 pad 2: GND -> Net-(D11-Pad2)
- RL4 pad 2: GND -> Net-(D12-Pad2)
- U4 pad 22: Pgood Vout -> EN_Vout
- U4 pad 24: EN_Vout -> SWCLK
- U5 pad 1: Vin -> V+
Routing:
- net Net-(D12-Pad2): track 0.00 -> 49.6 mm, vias 0 -> 1
- net Net-(D9-Pad2): track 0.00 -> 48.1 mm, vias 0 -> 1
- net Net-(D10-Pad2): track 0.00 -> 31.8 mm, vias 0 -> 1
- net Vin: track 265.5 -> 295.2 mm, vias 11 -> 14
- net Net-(D9-Pad1): track 46.2 -> 18.5 mm
- net Net-(D11-Pad2): track 0.00 -> 26.8 mm, vias 0 -> 1
- net SWCLK: track 0.00 -> 25.8 mm, vias 0 -> 3
- net Error: track 24.9 -> 44.8 mm, vias 2 -> 4
- net Net-(D11-Pad1): track 46.6 -> 30.8 mm
- net Net-(D10-Pad1): track 44.4 -> 28.6 mm
- net Net-(D12-Pad1): track 32.9 -> 19.2 mm
- net Relay1: track 55.5 -> 69.1 mm
- net Relay4: track 60.9 -> 73.2 mm
- net Relay2: track 62.3 -> 72.2 mm
- net Relay3: track 58.7 -> 67.9 mm, vias 2 -> 4
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Other:
- outline, holes or cut-outs redrawn
- board text added: "3.3V"
- board text added: "SCLK"
- board text added: "SWD"
