File: Powerboard 1/PowerBoard 1/PowerBoard 1.kicad_sch (KiCad schematic)
At the start: 155 parts, among them J1 Conn_01x03_Male, J2 Conn_01x03_Male, J3 Conn_01x03_Male, J4 Conn_01x03, J5 Conn_01x02_Male, J6 Conn_02x20_Counter_Clockwise, J7 Conn_01x01_Female, J8 Conn_01x01_Female, Q1 TP0610L, Q2 BC808, Q3 BC808, Q4 BC808, Q5 BC808, Q6 2N3904, Q7 2N3904, Q8 BC808, SW1 SW_Push, U1 ISO1540DR, U10 LM335Z, U11 TL062, U12 EL3H7-G, U13 EL3H7-G, U14 LT3083, U15 TL062, U16 LM334Z, U2 LT6657AHMS8-3, U3 LT8607, U4 STM32F303K8Tx, U5 LT3680, U6 M24C01-FDW, U7 LM334Z, U8 LM335Z, U9 LM334Z, Y1 8Mhz

Commit message: Rev 3 Pcb's
Parts:
- removed Q2, Q3, Q4, Q5: BC808, Package_TO_SOT_SMD:SOT-23, symbol Transistor_BJT:BC808
- added D10, D11, D12, D9: ss34, Diode_SMD:D_SMA_Handsoldering, symbol Device:D
- added J9: Conn_01x04, Connector_PinSocket_2.54mm:PinSocket_1x04_P2.54mm_Vertical, symbol Connector_Generic:Conn_01x04
- added Q2, Q3, Q4, Q5: 2N3904, Package_TO_SOT_SMD:SOT-23, symbol Transistor_BJT:2N3904
- added R10: 10Kohm, Resistor_SMD:R_0805_2012Metric_Pad1.20x1.40mm_HandSolder, symbol Device:R
- added R11, R12, R70: 20Kohm, Resistor_SMD:R_0805_2012Metric_Pad1.20x1.40mm_HandSolder, symbol Device:R
- added R71: 8Kohm, Resistor_SMD:R_0805_2012Metric_Pad1.20x1.40mm_HandSolder, symbol Device:R
- C1, C30: Orderd (none) -> 40
- C10, C23, C24, C26: Buylink C784103 -> C153034
- C11, C12: value 0.1µF -> 100nF
- C13, L1: Orderd (none) -> 30
- C16: value 1uF Film -> 1uF; Buylink C216548 -> C123629; Orderd (none) -> 100
- C17: Orderd (none) -> 50
- C18: Buylink C216548 -> C28323; Orderd (none) -> 100
- C2: Buylink C17024 -> C440198
- C20, D5, U12, U13: Orderd (none) -> 20
- C21, R49, R54, R69: Orderd (none) -> 100
- C22: value 0.47µF -> 470nF; Buylink C106843 -> C307545; Orderd (none) -> 100
- C27, C4: Buylink C72505 -> C98744
- C3: value 1pF -> 1uF
- C32, C35: Buylink C76651 -> C215908; Orderd (none) -> 100
- C34: Buylink C45783 -> C338080; Orderd (none) -> 10
- C36: value 1µ -> 1uF; Buylink C216548 -> C123629; Orderd (none) -> 100
- C38: Buylink C476766 -> C525005; Orderd (none) -> 20
- C6, C7: Buylink C94472 -> C309037
- C8: Buylink C77096 -> C513768; Orderd (none) -> 30
- C9: Buylink C83170 -> C780691; Orderd (none) -> 100
- D1: Buylink C134454 -> C433997; Orderd (none) -> 50
- D2, D3, D4, D6, D7, D8, L2, U1: Orderd (none) -> 10
- F1, F2, F3, F4, Y1: Orderd (none) -> 15
- J7, J8: Orderd (none) -> 6
- Q1: footprint Package_TO_SOT_THT:TO-92L_Inline -> Package_TO_SOT_SMD:SOT-23; Buylink C106271 -> C193222; Orderd (none) -> 10
- Q6, Q7: footprint Package_TO_SOT_THT:TO-92_Inline -> Package_TO_SOT_SMD:SOT-23; Orderd (none) -> 100
- R14: value 100Kohm -> 10K
- R2: Buylink (none) -> C168424; Orderd (none) -> 100
- R31, R45, R60: value 20Kohm -> 8Kohm; Orderd (none) -> 100
- R32, R48, R55, R64: value 370ohm -> 800ohm
- R33, R34, R35, R36, R37, R38, R39, R40, R41, R42: Buylink C514992 -> C304864; Orderd (none) -> 100
- R46: value 20Kohm -> 100Kohm; Orderd (none) -> 100
- R47: value 4Kohm -> 100Kohm; Buylink C88431 -> C413705; Orderd (none) -> 20
- R52: value 100Kohm 0.1% -> 20Kohm
- R6: Buylink C149966 -> C322296; Orderd (none) -> 100
- R7: Buylink C218655 -> C322540; Orderd (none) -> 100
- R8: Buylink C218502 -> C57148; Orderd (none) -> 100
- R9: Buylink C218408 -> C131391; Orderd (none) -> 100
- RL1, RL2, RL3, RL4: Orderd (none) -> 28
Connections:
- net +3V3: now also J9.1 (Pin_1)
- net EN_Vout: now also U4.22 (PA12); no longer U4.24 (PA14)
- net Error: now also J9.2 (Pin_2)
- net GND: now also R54.1, J9.4 (Pin_4), Q2.1 (E), Q3.1 (E), Q4.1 (E), Q5.1 (E), R11.1, R12.1, R70.1; no longer RL1.2 (L2), RL2.2 (L2), RL3.2 (L2), RL4.2 (L2)
- net Iout_ADC: now also U15.5 (+); no longer U15.6 (-)
- net Iout_DAC: now also U15.6 (-); no longer U15.5 (+)
- net Pgood Vout: now also R10.2; no longer U4.22 (PA12)
- net Relay1: now also R11.2
- net Relay2: now also R12.2
- net Relay3: now also R54.2, R60.1; no longer R54.1
- net Relay4: now also R70.2, R71.1; no longer R60.1
- net V+: now also U5.1 (BD)
- net Vin: now also R32.2, R48.2, R55.2, R64.2; no longer U5.1 (BD)
- net at R60.2: now also Q4.2 (B)
- net at R45.2: now also Q3.2 (B)
- net at R55.1, RL3.1 (L1): now also D11.1 (K)
- net at R31.2: now also Q2.2 (B)
- net at R64.1, RL4.1 (L1): now also D12.1 (K)
- net at R32.1, RL1.1 (L1): now also D9.1 (K)
- net at R48.1, RL2.1 (L1): now also D10.1 (K)
- new net: D11.2 (A), Q4.3 (C), RL3.2 (L2)
- new net: D10.2 (A), Q3.3 (C), RL2.2 (L2)
- new net: D9.2 (A), Q2.3 (C), RL1.2 (L2)
- new net: Q5.2 (B), R71.2
- new net: D12.2 (A), Q5.3 (C), RL4.2 (L2)
- new net SWCLK: J9.3 (Pin_3), R10.1, U4.24 (PA14)
Other:
- moved on the sheet: F2, F3, F4, J5, J6, J7, J8, Q8, R31, R32, R43, R44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

Commit message: Final Version Tested
Parts:
- removed C1, C30: 100µF, Capacitor_SMD:C_Elec_8x10.2, symbol Device:CP
- removed C10, C23, C24, C26: 22µF X7R, Capacitor_SMD:C_2220_5650Metric_Pad1.97x5.40mm_HandSolder, symbol Device:C
- removed C11, C38: 100nF, Capacitor_SMD:C_0805_2012Metric_Pad1.18x1.45mm_HandSolder, symbol Device:C
- removed C13: 10µF X7R, Capacitor_SMD:C_1206_3216Metric_Pad1.33x1.80mm_HandSolder, symbol Device:C
- removed C14: Optional, Capacitor_SMD:C_0805_2012Metric_Pad1.18x1.45mm_HandSolder, symbol Device:C
- removed C15, C19, C33, C37: Decoupling, Capacitor_SMD:C_0805_2012Metric_Pad1.18x1.45mm_HandSolder, symbol Device:C
- removed C17: 680pF, Capacitor_SMD:C_0805_2012Metric_Pad1.18x1.45mm_HandSolder, symbol Device:C
- removed C18: 1µF X7R, Capacitor_SMD:C_0805_2012Metric_Pad1.18x1.45mm_HandSolder, symbol Device:C
- removed C20: 0.1pF, Capacitor_SMD:C_0603_1608Metric_Pad1.08x0.95mm_HandSolder, symbol Device:C
- removed C21: 10pF, Capacitor_SMD:C_0805_2012Metric_Pad1.18x1.45mm_HandSolder, symbol Device:C
- removed C22: 470nF, Capacitor_SMD:C_0805_2012Metric_Pad1.18x1.45mm_HandSolder, symbol Device:C
- removed C27, C4: 22µF, Capacitor_SMD:C_Elec_6.3x5.4, symbol Device:CP
- removed C3, C36: 1uF, Capacitor_SMD:C_0805_2012Metric_Pad1.18x1.45mm_HandSolder, symbol Device:C
- removed C32, C35: 4.7µF, Capacitor_SMD:C_0805_2012Metric_Pad1.18x1.45mm_HandSolder, symbol Device:C
- removed C34: 22µF, Capacitor_SMD:C_0805_2012Metric_Pad1.18x1.45mm_HandSolder, symbol Device:C
- removed C8: 4.7µF X7R, Capacitor_SMD:C_1206_3216Metric_Pad1.33x1.80mm_HandSolder, symbol Device:C
- removed C9: 10nF, Capacitor_SMD:C_0805_2012Metric_Pad1.18x1.45mm_HandSolder, symbol Device:C
- removed D1: B340, Diode_SMD:D_SMA_Handsoldering, symbol Diode:B340
- removed D10, D11, D12, D9: ss34, Diode_SMD:D_SMA_Handsoldering, symbol Device:D
- removed D7, D8: MBRD1035CTL, Package_TO_SOT_SMD:TO-252-2, symbol Device:D_Schottky
- removed F1: 3,5A Polyfuse, Fuse:Fuse_1206_3216Metric_Pad1.42x1.75mm_HandSolder, symbol Device:Polyfuse
- removed F2, F4: 15A Polyfuse, Fuse:Fuse_1812_4532Metric_Pad1.30x3.40mm_HandSolder, symbol Device:Polyfuse
- removed J6: Conn_02x20_Counter_Clockwise, Connector_PinSocket_2.54mm:PinSocket_2x20_P2.54mm_Vertical, symbol Connector_Generic:Conn_02x20_Odd_Even
- removed L1: 2.2µF, Inductor_SMD:L_Wuerth_MAPI-3020, symbol Device:L
- removed L2: 4.7µH 5A, Inductor_SMD:L_7.3x7.3_H3.5, symbol Device:L
- removed Q1: TP0610L, Package_TO_SOT_SMD:SOT-23, symbol Transistor_FET:TP0610L
- removed Q2, Q3, Q4, Q5, Q6, Q7: 2N3904, Package_TO_SOT_SMD:SOT-23, symbol Transistor_BJT:2N3904
- removed Q8: BC808, Package_TO_SOT_SMD:SOT-23, symbol Transistor_BJT:BC808
- removed R1, R13, R46, R47: 100Kohm, Resistor_SMD:R_0805_2012Metric_Pad1.20x1.40mm_HandSolder, symbol Device:R
- removed R11, R12, R49, R52, R54, R69, R70: 20Kohm, Resistor_SMD:R_0805_2012Metric_Pad1.20x1.40mm_HandSolder, symbol Device:R
- removed R14: 10K, Resistor_SMD:R_0805_2012Metric_Pad1.20x1.40mm_HandSolder, symbol Device:R
- removed R17: 200Kohm, Resistor_SMD:R_0805_2012Metric_Pad1.20x1.40mm_HandSolder, symbol Device:R
- removed R18, R20, R21, R23, R24, R61, R62: 10Kohm, Resistor_SMD:R_0805_2012Metric_Pad1.20x1.40mm_HandSolder, symbol Device:R
- removed R19, R22, R56: 68ohm, Resistor_SMD:R_0805_2012Metric_Pad1.20x1.40mm_HandSolder, symbol Device:R
- removed R2: 18.2Kohm, Resistor_SMD:R_0805_2012Metric_Pad1.20x1.40mm_HandSolder, symbol Device:R
- removed R31, R45, R60, R71: 8Kohm, Resistor_SMD:R_0805_2012Metric_Pad1.20x1.40mm_HandSolder, symbol Device:R
- removed R32, R48, R55, R64: 800ohm, Resistor_SMD:R_0805_2012Metric_Pad1.20x1.40mm_HandSolder, symbol Device:R
- removed R33, R34, R35, R36, R37, R38, R39, R40, R41, R42: 2ohm, Resistor_SMD:R_0805_2012Metric_Pad1.20x1.40mm_HandSolder, symbol Device:R
- removed R43, R44, R50, R51: R, Resistor_SMD:R_0805_2012Metric_Pad1.20x1.40mm_HandSolder, symbol Device:R
- removed R53, R57, R63, R66: 1Kohm, Resistor_SMD:R_0805_2012Metric_Pad1.20x1.40mm_HandSolder, symbol Device:R
- removed R58, R59, R65, R67: 18Kohm, Resistor_SMD:R_0805_2012Metric_Pad1.20x1.40mm_HandSolder, symbol Device:R
- removed R6: 15.4Kohm, Resistor_SMD:R_0805_2012Metric_Pad1.20x1.40mm_HandSolder, symbol Device:R
- removed R68: 100ohm, Resistor_SMD:R_0805_2012Metric_Pad1.20x1.40mm_HandSolder, symbol Device:R
- removed R7: 63.4Kohm, Resistor_SMD:R_0805_2012Metric_Pad1.20x1.40mm_HandSolder, symbol Device:R
- removed R8: 309Kohm, Resistor_SMD:R_0805_2012Metric_Pad1.20x1.40mm_HandSolder, symbol Device:R
- removed R9: 1Mohm, Resistor_SMD:R_0805_2012Metric_Pad1.20x1.40mm_HandSolder, symbol Device:R
- removed RL1, RL2, RL3, RL4: JQC-3FF, 00_Custom_Kicad:JQC-3FF, symbol 00_LIB:JQC-3FF
- removed U1: ISO1540DR, Package_SO:SOIC-8_3.9x4.9mm_P1.27mm, symbol Isolator:ISO1541
- removed U10, U8: LM335Z, Package_TO_SOT_THT:TO-92_Inline, symbol 00_LIB:LM335Z
- removed U11, U15: TL062, Package_SO:SOIC-8_3.9x4.9mm_P1.27mm, symbol Amplifier_Operational:TL062
- removed U12, U13: EL3H7-G, Package_SO:SOP-4_4.4x2.6mm_P1.27mm, symbol 00_LIB:EL3H7-G
- removed U14: LT3083, Package_TO_SOT_THT:TO-220-5_Horizontal_TabDown, symbol 01-Global-LIB:LT3083
- removed U16, U7, U9: LM334Z, Package_TO_SOT_THT:TO-92_Inline, symbol Reference_Current:LM334Z
- removed U3: LT8607, 00_Custom_Kicad:MSOP-10_handsolder, symbol 00_LIB:LT8607
- removed U5: LT3680, 00_Custom_Kicad:MSOP-10_handsolder, symbol 01-Global-LIB:LT3680
Connections:
- no-connect marks 1 -> 0
Other:
- added sheet Buck converters (BuckConv.kicad_sch)
- added sheet Bussconnector + isolation (Buss.kicad_sch)
- added sheet Feedback (LDO.kicad_sch)
- added sheet PowerMatrix (PowerMatrix.kicad_sch)
- added sheet TempSens (TempSens.kicad_sch)
- note removed: "3.3V 500mA Buck converter"
- note removed: "Current Limter 0-3A 0-3V"
- note removed: "Current Sense IinLDO ~~ IoutLDO 0-3A 0-3V"
- note removed: "I2C Isolator"
- note removed: "Minimum load LM3083 1mA Const"
- note removed: "Opto isolator"
- note removed: "Output 3.5A Buck converter 1.8Mhz Swiching Freq"
- note removed: "Output Connectors"
- note removed: "Over Voltage Protection"
- note removed: "Supply OpAmps"
- note removed: "Temperature sensors"
- note removed: "Vbus Relais"
- note removed: "Voltage control 0-3V In"
- note removed: "Vout sense 0-30V 0-3Vout"
- note removed: "liniar voltage dropout and feedback 3A 0-20V"
- moved on the sheet: C12, C16, C2, C25, C28, C31, C5, C6, C7, D2, D3, D4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
