File: Controller/Controller/Controller/Controller.kicad_pcb (KiCad board)
At the start: 4 copper layers, 121 x 80 mm, 124 parts, among them J1 Conn_01x02, J2 Conn_02x20_Counter_Clockwise, J3 Conn_01x06, J4 Conn_01x05, J5 USB_A, J6 USB_C_Receptacle_USB2.0, J7 RJ45_Amphenol_RJMG1BD3B8K1ANR, J8 Conn_01x06_MountingPin, J9 Conn_01x50_MountingPin, Q1 CSD16323Q3, SW1 SW_Push, SW2 SW_Push, U1 STM32F746IGTx, U10 LTC1261L, U2 LAN8720A, U3 M24C02-WMN, U4 LM317_TO-252, U5 AMS1117-3.3, U6 LM317_TO-252, U7 LM3488, U8 C85037, U9 LM317_TO-252, X1 XO32, Y1 32.765Mhz

Commit message: contoller and contoller front Rev 1
Parts:
- removed R28: 10Kohm, Resistor_SMD:R_0805_2012Metric_Pad1.20x1.40mm_HandSolder
- removed the REF** at (71.0, 120.4)
- removed the REF** at (182.0, 120.5)
- removed the REF** at (78.5, 49.6)
- removed the REF** at (161.9, 49.6)
- added C50: 100uF, Capacitor_SMD:CP_Elec_5x5.4, F.Cu at (80.6, 40.8)
- added C51: 4.7uF, Capacitor_SMD:C_0805_2012Metric_Pad1.18x1.45mm_HandSolder, F.Cu at (80.0, 45.0)
- added R: MountingHole_3.2mm_M3_Pad_Via, MountingHole:MountingHole_3.2mm_M3_Pad_Via, F.Cu at (71.5, 119.5)
- added REF**: MountingHole_3.2mm_M3_Pad_Via, MountingHole:MountingHole_3.2mm_M3_Pad_Via, F.Cu at (71.5, 34.5)
- added REF**: MountingHole_3.2mm_M3_Pad_Via, MountingHole:MountingHole_3.2mm_M3_Pad_Via, F.Cu at (161.5, 119.5)
- added REF**: MountingHole_3.2mm_M3_Pad_Via, MountingHole:MountingHole_3.2mm_M3_Pad_Via, F.Cu at (161.5, 34.5)
- moved U9 118.7 mm to (82.8, 33.8), turned to 180 degrees
- moved R43 107.4 mm to (88.2, 39.8), turned to 0 degrees
- moved R44 103.1 mm to (88.2, 41.8)
- moved U6 90.0 mm to (96.8, 33.8)
- moved R33 87.0 mm to (121.4, 32.6), turned to 180 degrees
- moved R35 86.6 mm to (102.6, 41.8), turned to 180 degrees
- moved R34 83.9 mm to (102.6, 39.8)
- moved C30 82.7 mm to (125.4, 30.6), turned to 180 degrees
- moved C31 82.0 mm to (125.4, 32.6), turned to 180 degrees
- moved R41 81.0 mm to (123.6, 36.8)
- moved C49 80.4 mm to (94.2, 45.0), turned to 0 degrees
- moved C33 79.8 mm to (126.5, 38.0)
- moved R36 77.6 mm to (128.5, 38.0)
- moved U7 76.1 mm to (133.0, 32.0), turned to 0 degrees
- moved C48 74.4 mm to (94.6, 40.6), turned to 0 degrees
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Routing:
- net 9.6V: track 58.3 -> 177.9 mm
- net 18V: track 236.3 -> 288.9 mm, vias 4 -> 8
- net Net-(R8-Pad1): track 72.3 -> 40.0 mm, vias 4 -> 2
- net Net-(R9-Pad1): track 73.2 -> 41.4 mm, vias 4 -> 2
- net RMII_TXEN: track 81.3 -> 58.1 mm
- net RMII_RXER: track 73.8 -> 52.1 mm
- net RMII_RXD-: track 45.7 -> 25.8 mm
- net RMII_MDIO: track 37.3 -> 17.8 mm, vias 2 -> 0
- net RMII_REF_CLK: track 39.2 -> 19.7 mm, vias 2 -> 0
- net RMII_CRS_DV: track 43.6 -> 24.5 mm
- net RMII_RXD+: track 45.0 -> 26.3 mm
- net RMII_TXD+: track 68.1 -> 51.4 mm
- net RESET: track 55.3 -> 39.3 mm, vias 4 -> 3
- net RMII_TXD-: track 67.0 -> 52.9 mm
- net RMII_MDC: track 40.1 -> 26.0 mm
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Other:
- board size 121 x 80 mm -> 101 x 96 mm

Commit message: ReV 2 of the contoller Board
Parts:
- removed R: MountingHole_3.2mm_M3_Pad_Via, MountingHole:MountingHole_3.2mm_M3_Pad_Via
- removed the REF** at (71.5, 34.5)
- removed the REF** at (161.5, 119.5)
- removed the REF** at (161.5, 34.5)
- added C52: 100nF, Capacitor_SMD:C_0805_2012Metric_Pad1.18x1.45mm_HandSolder, F.Cu at (85.1, 63.8)
- added C53: 100nF, Capacitor_SMD:C_0805_2012Metric_Pad1.18x1.45mm_HandSolder, F.Cu at (85.5, 45.8)
- added C54: 100nF, Capacitor_SMD:C_0805_2012Metric_Pad1.18x1.45mm_HandSolder, F.Cu at (90.0, 63.2)
- added C55: 100nF, Capacitor_SMD:C_0805_2012Metric_Pad1.18x1.45mm_HandSolder, F.Cu at (72.4, 62.2)
- added C57: 100nF, Capacitor_SMD:C_0805_2012Metric_Pad1.18x1.45mm_HandSolder, F.Cu at (81.1, 62.5)
- added C58: 100nF, Capacitor_SMD:C_0805_2012Metric_Pad1.18x1.45mm_HandSolder, F.Cu at (74.5, 45.6)
- added J10: Conn_01x03, Connector_PinSocket_2.54mm:PinSocket_1x03_P2.54mm_Vertical, F.Cu at (136.1, 95.5)
- added R28: 10Kohm, Resistor_SMD:R_0805_2012Metric_Pad1.20x1.40mm_HandSolder, F.Cu at (109.0, 53.5)
- added REF**: MountingHole_3.5mm_Pad_Via, MountingHole:MountingHole_3.5mm_Pad_Via, F.Cu at (71.5, 34.5)
- added REF**: MountingHole_3.5mm_Pad_Via, MountingHole:MountingHole_3.5mm_Pad_Via, F.Cu at (161.5, 34.5)
- added REF**: MountingHole_3.5mm_Pad_Via, MountingHole:MountingHole_3.5mm_Pad_Via, F.Cu at (71.5, 119.5)
- added REF**: MountingHole_3.5mm_Pad_Via, MountingHole:MountingHole_3.5mm_Pad_Via, F.Cu at (161.5, 119.5)
- added U11: M13S128168A, Package_SO:TSOP-II-54_22.2x10.16mm_P0.8mm, F.Cu at (84.0, 53.8)
- moved R4 21.7 mm to (74.0, 66.5), turned to 90 degrees
- moved R3 14.2 mm to (79.9, 69.5)
- moved C10 3.20 mm to (100.4, 96.6), turned to 180 degrees
- moved R5 3.08 mm to (79.0, 84.7)
- moved R6 2.26 mm to (79.8, 87.5)
- moved C13 2.04 mm to (87.0, 74.7), turned to 90 degrees
- moved C14 1.84 mm to (86.9, 79.9), turned to 0 degrees
- moved C5 1.78 mm to (95.9, 63.2), turned to 90 degrees
- moved C7 1.64 mm to (101.1, 60.4)
- moved C9 1.34 mm to (108.2, 62.7)
- moved C2 1.15 mm to (93.9, 63.2)
- moved R20 0.98 mm to (128.8, 67.7)
- moved C3 0.75 mm to (89.0, 69.1)
- moved C41 0.53 mm to (121.9, 83.2)
- moved C47 0.30 mm to (83.3, 111.0)
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Connections:
- J2 pad 17: I2C1_SCL -> I2C4_SCL
- J2 pad 18: I2C1_SDA -> I2C4_SDA
- J2 pad 2: SPI1_MSIO -> SPI1_MISO
- J2 pad 8: SPI2_MSIO -> SPI2_MISO
- J9 pad 40: (no net) -> LCD_UPDN
- R5 pad 1: I2C1_SCL -> I2C4_SCL
- R6 pad 1: I2C1_SDA -> I2C4_SDA
- U1 pad 100: (no net) -> I2C4_SCL
- U1 pad 104: (no net) -> SDRAM_D0
- U1 pad 105: USER_BTN -> SDRAM_D1
- U1 pad 106: RMII_RXER -> (no net)
- U1 pad 108: (no net) -> SDRAM_BA0
- U1 pad 109: Galv_Interrupt -> SDRAM_BA1
- U1 pad 110: Galv_Enable -> LCD_R7
- U1 pad 112: (no net) -> SDRAM_SDCLK
- U1 pad 118: I2C3_SDA -> (no net)
- U1 pad 119: (no net) -> LCD_R6
- U1 pad 128: (no net) -> LCD_G2
- U1 pad 138: (no net) -> USER_BTN
- U1 pad 139: (no net) -> LCD_R2
- U1 pad 140: (no net) -> Galv_Enable
- U1 pad 141: (no net) -> Galv_Interrupt
- U1 pad 142: (no net) -> SDRAM_D2
- U1 pad 143: (no net) -> SDRAM_D3
- U1 pad 150: LCD_B2 -> UART_RX2
- U1 pad 152: (no net) -> LDC_MODE
- U1 pad 153: (no net) -> LCD_B2
- U1 pad 154: RMII_TXEN -> LCD_B3
- U1 pad 156: (no net) -> LCD_R0
- U1 pad 16: I2C2_SDA -> SDRAM_A0
- U1 pad 160: (no net) -> SDRAM_SDNCAS
- U1 pad 161: (no net) -> ADDR_LED2
- U1 pad 162: SPI1_MOSI -> (no net)
- U1 pad 163: SPI1_MSIO -> SPI1_MOSI
- U1 pad 164: I2C1_SCL -> (no net)
- U1 pad 166: (no net) -> Boot0
- U1 pad 168: I2C1_SDA -> LCD_B7
- U1 pad 169: (no net) -> SDRAM_NBL0
- U1 pad 17: I2C2_SCL -> SDRAM_A1
- U1 pad 170: (no net) -> SDRAM_NBL1
- U1 pad 173: (no net) -> LCD_B4
- U1 pad 176: LCD_B7 -> (no net)
- U1 pad 18: LCD_CT_RESET -> SDRAM_A2
- U1 pad 19: LCD_CT_INT -> SDRAM_A3
- U1 pad 2: (no net) -> LCD_UPDN
- U1 pad 20: LCD_DITHB -> SDRAM_A4
- U1 pad 21: LDC_MODE -> SDRAM_A5
- U1 pad 26: LCD_SHLR -> LCD_CT_RESET
- U1 pad 27: (no net) -> LCD_CT_INT
- U1 pad 32: LCD_R5 -> SDRAM_SDNWE
- U1 pad 34: SPI2_MSIO -> SDRAM_SDNE0
- U1 pad 35: SPI2_MOSI -> SDRAM_SDCKE0
- U1 pad 40: (no net) -> ADDR_LED1
- U1 pad 43: LCD_R0 -> (no net)
- U1 pad 45: (no net) -> I2C2_SCL
- U1 pad 46: (no net) -> I2C2_SDA
- U1 pad 47: UART_RX2 -> ADDR_LED4
- U1 pad 50: (no net) -> RMII_RXER
- U1 pad 52: LCD_G2 -> SPI1_MISO
- U1 pad 56: LCD_R3 -> (no net)
- U1 pad 57: LCD_R6 -> (no net)
- U1 pad 59: (no net) -> SDRAM_SDNRAS
- U1 pad 60: (no net) -> SDRAM_A6
- U1 pad 63: (no net) -> SDRAM_A7
- U1 pad 64: (no net) -> SDRAM_A8
- U1 pad 65: (no net) -> SDRAM_A9
- U1 pad 66: (no net) -> SDRAM_A10
- U1 pad 67: (no net) -> SDRAM_A11
- U1 pad 68: (no net) -> SDRAM_D4
- U1 pad 69: (no net) -> SDRAM_D5
- U1 pad 7: (no net) -> LCD_SHLR
- U1 pad 70: ADDR_LED1 -> SDRAM_D6
- U1 pad 73: (no net) -> SDRAM_D7
- U1 pad 74: ADDR_LED2 -> SDRAM_D8
- U1 pad 75: LCD_B4 -> SDRAM_D9
- U1 pad 76: ADDR_LED3 -> SDRAM_D10
- U1 pad 77: ADDR_LED4 -> SDRAM_D11
- U1 pad 78: LCD_R7 -> SDRAM_D12
- U1 pad 79: (no net) -> ADDR_LED3
- U1 pad 8: (no net) -> LCD_DITHB
- U1 pad 80: (no net) -> RMII_TXEN
- U1 pad 85: LCD_R2 -> I2C3_SDA
- U1 pad 86: (no net) -> LCD_R3
- U1 pad 88: (no net) -> LCD_R5
- U1 pad 89: (no net) -> I2C4_SDA
- U1 pad 94: (no net) -> SPI2_MISO
- U1 pad 95: (no net) -> SPI2_MOSI
- U1 pad 96: (no net) -> SDRAM_D13
- U1 pad 97: (no net) -> SDRAM_D14
- U1 pad 98: LCD_B3 -> SDRAM_D15
Routing:
- net SPI1_MSIO: track 75.6 -> 0.00 mm, vias 4 -> 0
- net SDRAM_NBL1: track 0.00 -> 60.0 mm, vias 0 -> 3
- net SDRAM_SDCLK: track 0.00 -> 52.0 mm, vias 0 -> 2
- net I2C1_SDA: track 51.9 -> 0.00 mm, vias 2 -> 0
- net SPI2_MSIO: track 51.4 -> 0.00 mm, vias 2 -> 0
- net SDRAM_NBL0: track 0.00 -> 51.4 mm, vias 0 -> 2
- net SPI1_MISO: track 0.00 -> 49.8 mm, vias 0 -> 2
- net I2C4_SDA: track 0.00 -> 49.5 mm, vias 0 -> 4
- net SDRAM_SDNWE: track 0.00 -> 49.3 mm, vias 0 -> 2
- net SDRAM_SDNE0: track 0.00 -> 49.3 mm, vias 0 -> 3
- net SDRAM_SDCKE0: track 0.00 -> 48.5 mm, vias 0 -> 2
- net SDRAM_D2: track 0.00 -> 47.8 mm, vias 0 -> 4
- net I2C1_SCL: track 47.7 -> 0.00 mm, vias 2 -> 0
- net SDRAM_D3: track 0.00 -> 46.8 mm, vias 0 -> 4
- net SDRAM_SDNCAS: track 0.00 -> 46.8 mm, vias 0 -> 2
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Other:
- board text added: "0"
- board text added: "1"
- board text added: "A"
- board text added: "B"
- board text added: "Boot"
- board text added: "Contoller By Arne Van den Broeck (Nortle) Rev 2"
- board text added: "Gnd Vin"
- board text removed: "encoder A"
- board text removed: "encoder B"

Commit message: Rev 3 Pcb's
Parts:
- removed C28: 330uF, Capacitor_SMD:CP_Elec_8x10
- removed C39: 270uF, Capacitor_SMD:CP_Elec_10x12.6
- removed C46, C50: 100uF, Capacitor_SMD:CP_Elec_5x5.4
- removed C47: 4.7uF, Capacitor_SMD:C_0805_2012Metric_Pad1.18x1.45mm_HandSolder
- removed L2: 1.8uH, Inductor_SMD:L_6.3x6.3_H3
- removed Q1: CSD16323Q3, Package_TO_SOT_SMD:TDSON-8-1
- removed REF** (x4): MountingHole_3.5mm_Pad_Via, MountingHole:MountingHole_3.5mm_Pad_Via
- removed U4: LM317_TO-252, Package_TO_SOT_SMD:TO-252-2
- removed U7: LM3488, Package_SO:MSOP-8_3x3mm_P0.65mm
- added C56: 100nF, Capacitor_SMD:C_0805_2012Metric_Pad1.18x1.45mm_HandSolder, F.Cu at (89.2, 30.5)
- added C59: 22uF, Capacitor_SMD:CP_Elec_3x5.3, F.Cu at (97.2, 36.0)
- added L3: 15uH, Inductor_SMD:L_10.4x10.4_H4.8, F.Cu at (81.5, 35.0)
- added R30: 27Kohm, Resistor_SMD:R_0805_2012Metric_Pad1.20x1.40mm_HandSolder, F.Cu at (97.2, 30.5)
- added R45: 68Kohm, Resistor_SMD:R_0805_2012Metric_Pad1.20x1.40mm_HandSolder, F.Cu at (109.2, 44.5)
- added R46: 130Kohm, Resistor_SMD:R_0805_2012Metric_Pad1.20x1.40mm_HandSolder, F.Cu at (119.5, 63.0)
- added R47: 15Kohm, Resistor_SMD:R_0805_2012Metric_Pad1.20x1.40mm_HandSolder, F.Cu at (119.5, 65.0)
- added R48: Optional, Resistor_SMD:R_0805_2012Metric_Pad1.20x1.40mm_HandSolder, F.Cu at (135.5, 119.5)
- added R49: Optional, Resistor_SMD:R_0805_2012Metric_Pad1.20x1.40mm_HandSolder, F.Cu at (129.0, 100.5)
- added R50: Optional, Resistor_SMD:R_0805_2012Metric_Pad1.20x1.40mm_HandSolder, F.Cu at (146.5, 108.0)
- added R51: Optional, Resistor_SMD:R_0805_2012Metric_Pad1.20x1.40mm_HandSolder, F.Cu at (129.0, 102.5)
- added U12: LM2931-ADJ_soic-8, Package_SO:SOIC-8_3.9x4.9mm_P1.27mm, F.Cu at (148.7, 48.5)
- C30: value 560pF -> 4.7uF
- C31: value 6.8nF -> 330uF; footprint Capacitor_SMD:C_0805_2012Metric_Pad1.18x1.45mm_HandSolder -> Capacitor_SMD:CP_Elec_10x10.5
- C33: value 10pF -> 330uF; footprint Capacitor_SMD:C_0805_2012Metric_Pad1.18x1.45mm_HandSolder -> Capacitor_SMD:CP_Elec_10x10.5
- C38: value 100uF -> 330uF; footprint Capacitor_SMD:CP_Elec_5x5.4 -> Capacitor_SMD:CP_Elec_10x10.5
- C45, C49, C51: value 4.7uF -> 100nF
- C48: value 100uF -> 3.3uF; footprint Capacitor_SMD:CP_Elec_5x5.4 -> Capacitor_SMD:CP_Elec_4x5.7
- R10: value a -> 100ohm
- R31: value 62Kohm -> RTRIM; footprint Resistor_SMD:R_0805_2012Metric_Pad1.20x1.40mm_HandSolder -> Potentiometer_SMD:Potentiometer_Bourns_3214J_Horizontal
- R32: value 47Kohm -> 10Kohm
- R34: value 4.75Kohm -> 62Kohm
- R35: value 1.5Kohm -> 10Kohm
- R36: value 100ohm -> 10Kohm
- R37: value 5mohm -> 13Kohm; footprint Resistor_SMD:R_2512_6332Metric_Pad1.40x3.35mm_HandSolder -> Resistor_SMD:R_0805_2012Metric_Pad1.20x1.40mm_HandSolder
- R41: value 1Kohm -> 180Kohm
- R42: value 13.3Kohm -> 12Kohm
- R43: value 147Kohm -> 11Kohm
- R44: value 21.5Kohm -> 130Kohm
- U11: value M13S128168A -> IS42S16400J
- U5: value AMS1117-3.3 -> BD00C0AWFP; footprint Package_TO_SOT_SMD:SOT-223-3_TabPin2 -> Package_TO_SOT_SMD:TO-252-5_TabPin3
- U6: value LM317_TO-252 -> LMR50410; footprint Package_TO_SOT_SMD:TO-252-2 -> Package_TO_SOT_SMD:TSOT-23-6_HandSoldering
- U9: value LM317_TO-252 -> BD00C0AWFP; footprint Package_TO_SOT_SMD:TO-252-2 -> Package_TO_SOT_SMD:TO-252-5_TabPin3
- X1: value XO32 -> XO25
- moved C38 83.4 mm to (125.2, 36.2), turned to 90 degrees
- moved C30 79.2 mm to (142.3, 108.0)
- moved J8 74.2 mm to (81.2, 107.8)
- moved C51 71.0 mm to (150.5, 37.0), turned to 90 degrees
- moved R36 70.6 mm to (91.2, 98.0), turned to 90 degrees
- moved R38 68.3 mm to (155.6, 109.2)
- moved U8 68.3 mm to (155.5, 104.5)
- moved C32 68.3 mm to (155.4, 112.0)
- moved D1 68.3 mm to (160.3, 109.0)
- moved R44 67.4 mm to (155.4, 47.5), turned to -90 degrees
- moved R43 67.3 mm to (155.4, 43.6), turned to -90 degrees
- moved U9 62.7 mm to (145.5, 36.0), turned to 90 degrees
- moved L1 61.3 mm to (157.2, 96.7), turned to 180 degrees
- moved R1 60.9 mm to (89.0, 113.2)
- moved R2 60.8 mm to (87.0, 112.0)
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Connections:
- C29 pad 1: Vin -> 18V
- C30 pad 1: Net-(C30-Pad1) -> -6V
- C31 pad 1: Net-(C30-Pad1) -> VLCD
- C31 pad 2: Net-(C31-Pad2) -> GND
- C32 pad 1: 18V -> Vin
- C33 pad 1: Net-(C33-Pad1) -> VLCD
- C34 pad 1: +5V -> 9.6V
- C38 pad 1: GND -> VLCD
- C38 pad 2: -6V -> GND
- C44 pad 1: LCD_VDD -> +5V
- C45 pad 1: LCD_VDD -> +5V
- C48 pad 1: +5V -> VLCD
- C49 pad 1: +5V -> VLCD
- D1 pad 1: 18V -> Vin
- D2 pad 1: 18V -> VLCD
- D2 pad 2: Net-(D2-Pad2) -> Vin
- R31 pad 1: 2.9V -> 9.6V
- R31 pad 2: Net-(R31-Pad2) -> 2.9V
- R32 pad 1: Net-(R31-Pad2) -> 2.9V
- R33 pad 1: Net-(C31-Pad2) -> Power2
- R34 pad 1: +5V -> Net-(R30-Pad2)
- R34 pad 2: Net-(R34-Pad2) -> GND
- R35 pad 1: Net-(R34-Pad2) -> Power3
- R36 pad 1: Net-(R36-Pad1) -> Backlight
- R36 pad 2: Net-(C33-Pad1) -> GND
- R37 pad 1: Net-(C33-Pad1) -> 18V
- R37 pad 2: GND -> Net-(R37-Pad2)
- R38 pad 1: 18V -> Vin
- R41 pad 1: Net-(R41-Pad1) -> Net-(R37-Pad2)
- R42 pad 1: Net-(R41-Pad1) -> +5V
- R42 pad 2: 18V -> Net-(R42-Pad2)
- U1 pad 43: (no net) -> Vinsense
- U1 pad 56: (no net) -> Power3
- U1 pad 57: (no net) -> Power2
- U10 pad 1: +5V -> 9.6V
- U5 pad 1: GND -> Vin
- U5 pad 2: LCD_VDD -> Vin
- U5 pad 3: 18V -> GND
- U6 pad 1: Net-(R34-Pad2) -> Net-(C56-Pad2)
- U6 pad 2: +5V -> GND
- U6 pad 3: 18V -> Net-(R30-Pad2)
- U8 pad 5: 18V -> Vin
- U9 pad 1: Net-(R43-Pad2) -> Power2
- U9 pad 2: 9.6V -> VLCD
- U9 pad 3: 18V -> GND
Routing:
- net Vin: track 38.6 -> 170.5 mm, vias 0 -> 4
- net 18V: track 288.9 -> 157.6 mm, vias 8 -> 3
- net VLCD: track 0.00 -> 90.2 mm, vias 0 -> 2
- net +5V: track 269.8 -> 180.4 mm, vias 5 -> 3
- net Backlight: track 24.4 -> 109.5 mm, vias 4 -> 6
- net Power2: track 0.00 -> 67.4 mm, vias 0 -> 5
- net Power3: track 0.00 -> 63.5 mm, vias 0 -> 4
- net LCD_CT_INT: track 56.1 -> 118.0 mm
- net LCD_CT_RESET: track 52.8 -> 113.7 mm
- net LCD_VDD: track 264.9 -> 229.3 mm, vias 40 -> 42
- net GND: track 260.8 -> 296.1 mm, vias 67 -> 75
- net -6V: track 25.3 -> 51.4 mm
- net I2C3_SDA: track 97.3 -> 73.8 mm, vias 4 -> 2
- net I2C3_SCL: track 97.3 -> 74.6 mm, vias 2 -> 4
- net LCD_DEN: track 64.6 -> 43.4 mm
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
Commit message: Final Version Tested
Parts:
- removed R33, R35: 10Kohm, Resistor_SMD:R_0805_2012Metric_Pad1.20x1.40mm_HandSolder
- removed R46: 130Kohm, Resistor_SMD:R_0805_2012Metric_Pad1.20x1.40mm_HandSolder
- removed R47: 15Kohm, Resistor_SMD:R_0805_2012Metric_Pad1.20x1.40mm_HandSolder
- removed R48, R49, R50, R51: Optional, Resistor_SMD:R_0805_2012Metric_Pad1.20x1.40mm_HandSolder
- J1: value Conn_01x02 -> Power In
- J10: value Conn_01x03 -> Boot Select
- J2: value Conn_02x20_Counter_Clockwise -> Module Bus
- J3: value Conn_01x06 -> Programming Header
- J4: value Conn_01x05 -> Encoder Header
Connections:
- C34 pad 1: 9.6V -> +5V
- J9 pad 8: LCD_DEN -> LDC_MODE
- J9 pad 9: LDC_MODE -> LCD_DEN
- U1 pad 43: Vinsense -> (no net)
- U1 pad 56: Power3 -> (no net)
- U1 pad 57: Power2 -> (no net)
- U10 pad 1: 9.6V -> +5V
- U12 pad 5: Power3 -> (no net)
- U9 pad 1: Power2 -> (no net)
Routing:
- net +5V: track 180.4 -> 216.2 mm, vias 3 -> 4
- net 9.6V: track 193.6 -> 168.0 mm, vias 4 -> 2
- net Vin: track 170.5 -> 152.7 mm, vias 4 -> 3
- net 18V: track 157.6 -> 141.2 mm, vias 3 -> 2
- net GND: track 296.1 -> 282.3 mm, vias 75 -> 71
- net 2.9V: track 57.0 -> 47.3 mm
- net Power2: track 67.4 -> 58.2 mm
- net Vinsense: track 8.05 -> 0.00 mm, vias 2 -> 0
- net Power3: track 63.5 -> 60.4 mm, vias 4 -> 3
- net -6V: track 51.4 -> 49.2 mm
- net LDC_MODE: track 42.2 -> 42.9 mm
